Commit message: Add ARX deployment project
Include UMI policy inference scripts, ARX5 SDK changes, robot model files, and deployment documentation. Exclude local checkpoints, datasets, and evaluation outputs from the repository.

File: umi-deploy/arx5-sdk/models/L5_umi.urdf (robot description, URDF)
Before this commit: robot L5_umi, 8 links, 7 joints
Links:
- link base_link: geometry collision mesh filename=meshes/L5_umi/arm/raw_meshes_ARM/base_link_arm.STL; visual mesh filename=meshes/L5_umi/arm/raw_meshes_ARM/base_link_arm.STL
- link link1: geometry collision mesh filename=meshes/L5_umi/arm/raw_meshes_ARM/link1.STL; visual mesh filename=meshes/L5_umi/arm/raw_meshes_ARM/link1.STL
- link link2: geometry collision mesh filename=meshes/L5_umi/arm/raw_meshes_ARM/link2.STL; visual mesh filename=meshes/L5_umi/arm/raw_meshes_ARM/link2.STL
- link link3: geometry collision mesh filename=meshes/L5_umi/arm/raw_meshes_ARM/link3.STL; visual mesh filename=meshes/L5_umi/arm/raw_meshes_ARM/link3.STL
- link link4: geometry collision mesh filename=meshes/L5_umi/arm/raw_meshes_ARM/link4.STL; visual mesh filename=meshes/L5_umi/arm/raw_meshes_ARM/link4.STL
- link link5: geometry collision mesh filename=meshes/L5_umi/arm/raw_meshes_ARM/link5.STL; visual mesh filename=meshes/L5_umi/arm/raw_meshes_ARM/link5.STL
- link link6: geometry collision mesh filename=meshes/DAS_Controller_v3_r5_end_adapter_flange.STL scale=0.001 0.001 0.001; collision mesh filename=meshes/L5_umi/arm/raw_meshes_ARM/link6.STL
Joints:
- joint gripper_fixed_joint: origin xyz=0.235 0.0 0.0 rpy=0 0 0 -> xyz=0.0999414 0.0000388 0.0767217 rpy=0 0.2618 0

Commit message: Add ARX5 gravity compensation and improve runtime control

File: umi-deploy/arx5-sdk/models/L5_umi.urdf (robot description, URDF)
Before this commit: robot L5_umi, 8 links, 7 joints
Links:
- added link world
Joints:
- added joint world_to_base_link: type fixed, parent world, child base_link, origin xyz=0 0 0 rpy=0 0 0

Commit message: Update L5 UMI flange visualization

File: umi-deploy/arx5-sdk/models/L5_umi.urdf (robot description, URDF)
Before this commit: robot L5_umi, 9 links, 8 joints
Links:
- link link6: geometry collision mesh filename=meshes/DAS_Controller_v3_r5_end_adapter_flange.STL scale=0.001 0.001 0.001; collision mesh filename=meshes/L5_umi/umi/base_link.STL

Commit message: deploy R5 UMI model with LeRobot DiT policy compatibility

File: umi-deploy/arx5-sdk/models/L5_umi.urdf (robot description, URDF)
Before this commit: robot L5_umi, 9 links, 8 joints
Links:
- link base_link: geometry collision mesh filename=meshes/L5_umi/arm/base_link.STL; visual mesh filename=meshes/L5_umi/arm/base_link.STL
- link link1: mass 0.09728 -> 0.096804; geometry collision mesh filename=meshes/L5_umi/arm/link1.STL; visual mesh filename=meshes/L5_umi/arm/link1.STL
- link link2: mass 1.1477 -> 1.1988; geometry collision mesh filename=meshes/L5_umi/arm/link2.STL; visual mesh filename=meshes/L5_umi/arm/link2.STL
- link link3: mass 0.66 -> 0.84082; geometry collision mesh filename=meshes/L5_umi/arm/link3.STL; visual mesh filename=meshes/L5_umi/arm/link3.STL
- link link4: mass 0.11714 -> 0.12432; geometry collision mesh filename=meshes/L5_umi/arm/link4.STL; visual mesh filename=meshes/L5_umi/arm/link4.STL
- link link5: mass 0.6353 -> 0.63601; geometry collision mesh filename=meshes/L5_umi/arm/link5.STL; visual mesh filename=meshes/L5_umi/arm/link5.STL
- link link6: mass 0.902 -> 0.775
Joints:
- joint gripper_fixed_joint: origin xyz=0.0999414 0.0000388 0.0767217 rpy=0 0.2618 0 -> xyz=0.1039414 0.0000388 0.0767217 rpy=0 0.2618 0
- joint joint3: origin xyz=-0.264 0 0 rpy=3.1416 0 0 -> xyz=-0.264 0 0 rpy=-3.1416 0 0
- joint joint4: origin xyz=0.245 0 -0.06 rpy=0 0 0 -> xyz=0.245 -5E-05 -0.06 rpy=0 0 0
- joint joint5: origin xyz=0.06775 -5E-05 -0.0865 rpy=0 0 0 -> xyz=0.073914 5E-05 -0.083391 rpy=0 0 0
- joint joint6: origin xyz=0.02895 0 0.0865 rpy=3.1416 0 0 -> xyz=0.025286 0 0.083391 rpy=3.1416 0 0
